Commit message: finished chapter 3

File: mastering_ros_robot_description_pkg/urdf/pan_tilt.urdf (robot description, URDF)
Before this commit: robot pan_tilt, 3 links, 2 joints
Links:
- link base_link: mass None -> 1; geometry collision cylinder length=0.03 radius=0.2; visual cylinder length=0.01 radius=0.2
- link pan_link: mass None -> 1; geometry collision cylinder length=0.4 radius=0.06; visual cylinder length=0.4 radius=0.04
- link tilt_link: mass None -> 1; geometry collision cylinder length=0.4 radius=0.06; visual cylinder length=0.4 radius=0.04
Joints:
- joint tilt_joint: limit lower=-3.14 upper=3.14 effort=300 velocity=0.1 -> lower=-4.64 upper=-1.5 effort=300 velocity=0.1

File: mastering_ros_robot_description_pkg/urdf/sensors/xtion_pro_live.urdf.xacro (robot description, xacro)
@@ -1,4 +1,4 @@
 <?xml version="1.0"?>
-<robot xmlns:xacro="http://www.ros.org/wiki/xacro">
+<robot xmlns:xacro="http://ros.org/wiki/xacro">
   <xacro:include filename="$(find mastering_ros_robot_description_pkg)/urdf/sensors/xtion_pro_live.gazebo.xacro"/>
   <xacro:macro name="dummy_inertial">
@@ -40,5 +40,5 @@
     </joint>
     <link name="${name}_optical_frame">
-      <xacro:dummy_inertial/>
+      <dummy_inertial/>
     </link>
     <!-- Depth sensor frames -->
@@ -49,5 +49,5 @@
     </joint>
     <link name="${name}_depth_frame">
-      <xacro:dummy_inertial/>
+      <dummy_inertial/>
     </link>
     <joint name="${name}_depth_optical_joint" type="fixed">
@@ -57,5 +57,5 @@
     </joint>
     <link name="${name}_depth_optical_frame">
-      <xacro:dummy_inertial/>
+      <dummy_inertial/>
     </link>
     <!-- RGB sensor frames -->
@@ -66,5 +66,5 @@
     </joint>
     <link name="${name}_rgb_frame">
-      <xacro:dummy_inertial/>
+      <dummy_inertial/>
     </link>
     <joint name="${name}_rgb_optical_joint" type="fixed">
@@ -74,5 +74,5 @@
     </joint>
     <link name="${name}_rgb_optical_frame">
-      <xacro:dummy_inertial/>
+      <dummy_inertial/>
     </link>
     <xacro:xtion_pro_live_rgbd_camera_gazebo name="${name}"/>

File: mastering_ros_robot_description_pkg/urdf/seven_dof_arm.xacro (robot description, xacro)
@@ -406,7 +406,7 @@
   <!-- Define arm with gripper mounted on a base -->
   <!--
-  <xacro:base name="base" />
-  <xacro:arm name="arm" parent="base"/>
-  <xacro:gripper2 name="gripper2" parent="tool"/>
+  <xacro:base name="base"/>
+  <xacro:arm parent="base"/>
+  <xacro:gripper parent="tool"/>
 -->
   <!-- Define RGB-D sensor -->
